File: Hardware/HABEXpico8/HABEXpico8.brd (EAGLE design)
At the start: 160 x 100 mm, 48 parts, among them Q1 2.5A/30V, SW1 SKQGADE010, SW2 SKQGADE010, U1 LTC3106, U2 EVA-8M, U3 STM32L011G4, U4 3.3V, Y1 ABS07-120-32.768KHZ-T

Commit message: Updated Power System, detailed GPS and MCU
Updated Power System, detailed GPS and MCU, removed backup files.
Parts:
- removed U$1: JTI_ANTENNA-1575AT43A40, habexpico8:JTI_ANTENNA-1575AT43A40
- added C16: 0.1uF, SparkFun-Capacitors:0603
- added C17, C18: 6pF, rcl:C0603
- added C19: 1.0uF, SparkFun-Capacitors:0603
- added C20: 10nF, SparkFun-Capacitors:0603
- added C21: 10uF, SparkFun-Capacitors:0603
- added C22: 10uF, SparkFun-Capacitors:0805
- added CR2: USBLC6-2SC6, habexpico8:SOT23-6L
- added IC1: LT1763CS8-3.3, linear-technology:SOIC8
- added JP10, JP11, JP12, JP13, JP6, JP7, JP8, JP9: (no value), SparkFun-Retired:1X02
- added JP14, JP15, JP4, JP5: JUMPER-SMT_2_NO_SILK, SparkFun-Jumpers:SMT-JUMPER_2_NO_SILK
- added L2: 33nH/±5%/500mA, SparkFun-Coils:0603
- added R11: 10, SparkFun-Resistors:1206
- added R12: 10k, SparkFun-Resistors:0603
- added R13, R16: 27, SparkFun-Resistors:0603
- added R14, R15: 5.1k 10%, SparkFun-Resistors:0603
- added U5: USB-C_R/A_HYBRID_RCPT, habexpico8:USB-C_R/A_HYBRID_RCPT
- added U6: FT232RL, SparkFun-IC-Comms:SSOP28DB
- added X1, X2, X3, X4: BU-SMA-V, con-coax:BU-SMA-V
- added X5: JTI_ANTENNA-1575AT43A40, habexpico8:JTI_ANTENNA-1575AT43A40
- added X6: C-GRID-04-70553, con-molex:70553-04
- added X7: C-GRID-02-70553, con-molex:70553-02
- added Y2: ABS07-120-32.768KHZ-T, SparkFun-Clocks:CRYSTAL-SMD-3.2X1.5MM
- L1: value INDUCTOR-1210 -> 10uH
- moved JP2 197.4 mm to (-39.5, 96.3)
- moved JP3 197.4 mm to (-39.5, 77.5)
- moved R10 166.1 mm to (-14.1, 30.5)
- moved R9 150.6 mm to (-14.1, 18.2)
- moved J4 147.2 mm to (-28.8, 2.03)
- moved R4 2.01 mm to (27.1, 23.1)
Connections:
- net +5V renamed USB_VBUS
- new net 5V: C19.1, IC1.5, IC1.8, JP12.1, JP13.1
- new net AGND: U6.25
- new net GND18: U6.18
- new net GND21: U6.21
- new net GND7: U6.7
- new net N$12: C16.1, L2.1, R11.1
- new net N$13: C18.1, JP4.2, Y2.P$2
- new net N$14: L2.2, X2.1, X3.1
- new net N$15: CR2.6, R13.1
- new net N$16: CR2.4, R16.1
- new net N$19: C20.2, IC1.4
- new net REG_3.3V: C20.1, C21.1, IC1.1, IC1.2, JP11.2
- new net RF_IN: U2.1, X1.1
- new net SER_DN: R13.2
- new net SER_DP: R16.2
- new net USBC_CC1: R14.2, U5.A5
- new net USBC_CC2: R15.2, U5.B5
- new net USBC_DN: CR2.1, U5.A7, U5.B7
- new net USBC_DP: CR2.3, U5.A6, U5.B6
- new net USBC_GND: JP14.1, U5.A1, U5.A12, U5.B1, U5.B12, U5.SHL1, U5.SHL2, U5.SHL3, U5.SHL4
- new net USBC_VBUS: C22.1, CR2.5, JP12.2, U5.A4, U5.A9, U5.B4, U5.B9
- new net USB_GND: J2.GND1, J2.SHLD1, J2.SHLD2, J2.SHLD3, JP15.1
- new net VAUX_3.3V: JP10.2, X7.2
- new net VAUX_5V: JP13.2, X6.3, X6.4
- new net VCCIO: U6.4
- new net VSOLAR: C7.1, JP1.2, R1.2, SC1.1, SC2.1
- net 3.3V: now also J3.8, J4.8, JP10.1, JP11.1, R11.2, R12.2; no longer J3.6
- net GND: now also C16.2, C17.2, C18.2, C19.2, C21.2, C22.2, CR2.2, IC1.3, IC1.6, IC1.7, JP14.2, JP15.2, R14.1, R15.1, X1.2, X1.3, X1.4, X1.5, X2.2, X2.3, X2.4, X2.5, X3.2, X3.3, X3.4, X3.5, X4.2, X4.3, X4.4, X4.5, X6.1, X6.2, X7.1; no longer J2.GND1, J2.SHLD1, J2.SHLD2, J2.SHLD3
- net GPS_EN: now also J4.5
- net GPS_RESET: now also J4.2, R12.1; no longer J4.4
- net GPS_RX: now also J4.3; no longer J4.2
- net GPS_TX: now also J4.4; no longer J4.3
- net MCU_OSC32_IN: now also JP5.1
- net MCU_OSC32_OUT: now also JP4.1
- net N$10: now also C17.1, JP5.2, Y2.P$1; no longer JP1.1, U1.16
- net N$4: now also X4.1, X5.FEED; no longer U$1.FEED, U2.1
- net VCC: now also U6.20
- net VIN: now also JP1.1, U1.16; no longer C7.1, JP1.2, R1.2, SC1.1, SC2.1

Commit message: Added RF Front End w/ Simulation
Added RF Front End w/ Simulation
Parts:
- removed U$2: SI4464, habexpico8:QFN20+GNDPAD
- added C0: 43pF, Nordic_nRF:RESC0603_L
- added C23, C24, C27: 0.1uF, SparkFun-Capacitors:0603
- added C25: 10uF, SparkFun-Capacitors:0603
- added C26: 10nF, SparkFun-Capacitors:0603
- added C28, C29: 10pF, SparkFun-Capacitors:0603
- added C32: 15pF, Nordic_nRF:RESC0603_L
- added C33, CM1: 8.2pF, Nordic_nRF:RESC0603_L
- added D3: RED, SparkFun-LED:LED-0603
- added D4: GREEN, SparkFun-LED:LED-0603
- added JP16, JP17, JP18, JP19, JP20: JUMPER-3PTH, SparkFun-Retired:1X03
- added L5, L6, LM1: 18nH, Nordic_nRF:RESC0603_L
- added LC: 470nH, Nordic_nRF:RESC0603_L
- added R17, R18: 300, SparkFun-Resistors:0603
- added R19: 10k, SparkFun-Resistors:0603
- added R20, R21: 100k, SparkFun-Resistors:0603
- added SJ1, SJ2, SJ3, SJ4: SOLDERJUMPERNO, SparkFun-Retired:SJ_2S-NO
- added TP1, TP2: TPPAD1-13, testpad:P1-13
- added U7: 3.3V, SparkFun-IC-Power:SOT23-5
- added X8: 30MHZ 402F3001XIAR, IQD-Frequency-Products:2.0X1.6-4-PAD
- added X9: BU-SMA-V, con-coax:BU-SMA-V
- JP14, JP15: value JUMPER-SMT_2_NO_SILK -> JUMPER-3PTH; device SparkFun-Jumpers:SMT-JUMPER_2_NO_SILK -> SparkFun-Retired:1X03
- JP6, JP7, JP8, JP9: value (none) -> JUMPER-3PTH; device SparkFun-Retired:1X02 -> SparkFun-Retired:1X03
- U4: value 3.3V -> SI4464; device SparkFun-IC-Power:SOT23-5 -> habexpico8:QFN20+GNDPAD
- moved R13 406.2 mm to (-158.0, 138.2)
- moved U6 406.2 mm to (-154.2, 127.9)
- moved R16 406.2 mm to (-158.0, 134.9)
- moved JP14 279.1 mm to (-162.9, 14.5)
- moved JP15 259.9 mm to (-162.9, -4.32)
- moved JP6 167.6 mm to (-162.9, 89.7)
- moved JP7 167.6 mm to (-162.9, 70.9)
- moved U4 126.2 mm to (69.0, 39.4)
- moved JP8 75.0 mm to (-162.9, 52.1)
- moved JP9 75.0 mm to (-162.9, 33.3)
Connections:
- removed net AGND: U6.25
- removed net GND18: U6.18
- removed net GND21: U6.21
- removed net GND7: U6.7
- removed net USBC_GND: JP14.1, U5.A1, U5.A12, U5.B1, U5.B12, U5.SHL1, U5.SHL2, U5.SHL3, U5.SHL4
- removed net USB_GND: J2.GND1, J2.SHLD1, J2.SHLD2, J2.SHLD3, JP15.1
- removed net VCCIO: U6.4
- new net FTDI_SER_RXD: JP9.1, U6.5
- new net FTDI_SER_TXD: JP8.1, U6.1
- new net LPUART1_RX: JP6.2, JP6.3, U3.9
- new net LPUART1_TX: JP7.2, JP7.3, U3.8
- new net MCU_RADIO_EN: JP20.2, JP20.3, U3.18
- new net MCU_RADIO_GPIO1: JP19.2, JP19.3, U3.15
- new net MCU_RADIO_NIRQ: JP18.2, JP18.3, U3.14
- new net N$17: D3.C, U6.23
- new net N$18: D4.C, U6.22
- new net N$20: D3.A, R17.1
- new net N$21: D4.A, R18.1
- new net N$22: SJ1.2, U6.4
- new net N$23: R17.2, SJ2.1
- new net N$24: R18.2, SJ3.1
- new net N$25: R11.2, SJ4.1
- new net N$26: C28.1, TP1.TP, U4.17, X8.3
- new net N$27: C29.1, TP2.TP, U4.16, X8.1
- new net N$28: C0.1, LC.2, U4.4
- new net N$29: CM1.1, L5.2, LM1.1
- new net N$30: C0.2, LM1.2
- new net N$31: C32.1, L5.1, L6.2
- new net RADIO_EN: JP20.1, R21.1, U4.1
- new net RADIO_GPIO1: JP19.1, R20.1, U4.10
- new net RADIO_MISO: JP16.1, U4.13
- new net RADIO_MOSI: JP17.1, U4.14
- new net RADIO_NIRQ: JP18.1, U4.11
- new net RADIO_NSS: JP14.1, U4.15
- new net RADIO_SCLK: JP15.1, U4.12
- new net RF_OUT: C33.1, L6.1, X9.1
- new net SPI1_MISO: JP16.2, JP16.3, U3.12
- new net SPI1_MOSI: JP17.2, JP17.3, U3.13
- new net SPI1_NSS: JP14.2, JP14.3, U3.10
- new net SPI1_SCK: JP15.2, JP15.3, U3.11
- new net USART2_RX: JP8.2, JP8.3, U3.20
- new net USART2_TX: JP9.2, JP9.3, U3.19
- net 3.3V: now also C23.1, C25.1, C26.1, C27.1, LC.1, R20.2, R21.2, SJ1.1, SJ2.2, SJ3.2, SJ4.2, SW1.2, U4.6, U4.8; no longer R11.2
- net GND: now also C23.2, C24.2, C25.2, C26.2, C27.2, C28.2, C29.2, C32.2, C33.2, CM1.2, J2.GND1, J2.SHLD1, J2.SHLD2, J2.SHLD3, R14.2, R15.2, R19.1, U4.18, U4.21, U5.A1, U5.A12, U5.B1, U5.B12, U5.SHL1, U5.SHL2, U5.SHL3, U5.SHL4, U6.18, U6.21, U6.25, U6.26, U6.7, U7.2, X9.2, X9.3, X9.4, X9.5; no longer JP14.2, JP15.2, R14.1, R15.1, SW1.4, U4.2
- net GPS_EN: now also U3.7
- net GPS_RX: now also JP7.1
- net GPS_TX: now also JP6.1
- net GPS_USB_VDD: now also U7.5; no longer U4.5
- net MCU_RESET: now also R19.2, SW1.4; no longer SW1.2
- net SER_DN: now also U6.16
- net SER_DP: now also U6.15
- net USBC_CC1: now also R14.1; no longer R14.2
- net USBC_CC2: now also R15.1; no longer R15.2
- net USBC_VBUS: now also C24.1, U6.20
- net USB_VBUS: now also U7.1, U7.3; no longer U4.1, U4.3
- net VCC: no longer U6.20

Commit message: Finished schematic and simulations
Finished schematic and simulations. Expecting to make small tweaks in
future revisions.
Parts:
- removed C32: 15pF, Nordic_nRF:RESC0603_L
- removed C33, CM1: 8.2pF, Nordic_nRF:RESC0603_L
- removed L5, L6, LM1: 18nH, Nordic_nRF:RESC0603_L
- added CM: 4.7pF, Nordic_nRF:RESC0603_L
- added CM2: 7.5pF, Nordic_nRF:RESC0603_L
- added CX: 10pF, Nordic_nRF:RESC0603_L
- added J5: (no value), SparkFun-Connectors:1X08
- added L0: 56nH, Nordic_nRF:RESC0603_L
- added LM: 12nH, Nordic_nRF:RESC0603_L
- added LX: 140nH, Nordic_nRF:RESC0603_L
- C0: value 43pF -> 22pF
- moved IC1 208.0 mm to (57.9, 25.7)
- moved X7 204.7 mm to (77.2, 91.6)
- moved C0 194.5 mm to (-227.1, 58.7)
- moved C19 194.5 mm to (-182.5, 131.6)
- moved C20 194.5 mm to (-182.5, 128.3)
- moved C21 194.5 mm to (-182.5, 125.0)
- moved C28 194.5 mm to (-214.6, 91.3)
- moved JP18 194.5 mm to (-219.8, 36.4)
- moved LC 194.5 mm to (-227.1, 74.4)
- moved R14 194.5 mm to (-185.8, 113.4)
- moved R20 194.5 mm to (-214.6, 132.8)
- moved R21 194.5 mm to (-214.6, 122.9)
- moved TP1 194.5 mm to (-218.4, 91.3)
- moved TP2 194.5 mm to (-218.3, 88.1)
- moved X8 194.5 mm to (-211.2, 95.5)
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Connections:
- removed net RF_OUT: C33.1, L6.1, X9.1
- new net ANT_OUT: CM2.1, LM.1, X9.1
- net 3.3V: now also J5.8
- net GND: now also CM.2, CM2.2, CX.2, J5.1; no longer C32.2, C33.2, CM1.2
- net N$29: now also L0.1, LX.2; no longer CM1.1, L5.2, LM1.1
- net N$30: now also L0.2; no longer LM1.2
- net N$31: now also CM.1, CX.1, LM.2, LX.1; no longer C32.1, L5.1, L6.2
- net RADIO_EN: now also J5.2
- net RADIO_GPIO1: now also J5.3
- net RADIO_NIRQ: now also J5.4

Commit message: Added BOM, updated board/schematic files
Added BOM, updated board/schematic files
Parts:
- added JP21, JP22: (no value), SparkFun-Retired:1X03
- IC1: value LT1763CS8-3.3 -> (none)
- JP14, JP15, JP16, JP17, JP18, JP19, JP20, JP6, JP7, JP8, JP9: value JUMPER-3PTH -> (none)
- JP4, JP5: value JUMPER-SMT_2_NO_SILK -> (none)
- R1, R9: value 2.21M -> 1M
- R10, R2: value 1.33M -> 1M
- R14, R15: value 5.1k 10% -> 5.1K
- R3: value 10M -> 1M
- SJ1, SJ2, SJ3, SJ4: value SOLDERJUMPERNO -> (none)
- X1, X2, X3, X4, X9: value BU-SMA-V -> (none)
- Y1, Y2: value ABS07-120-32.768KHZ-T -> 32.768kHz
- moved JP20 275.9 mm to (49.4, 59.3), turned to 180 degrees
- moved JP19 272.0 mm to (49.4, 56.5), turned to 180 degrees
- moved J5 271.8 mm to (18.4, 86.4)
- moved JP18 269.8 mm to (49.4, 53.7), turned to 180 degrees
- moved C20 269.4 mm to (72.0, 40.0), turned to 180 degrees
- moved C19 268.2 mm to (72.0, 47.1), turned to 180 degrees
- moved C21 267.8 mm to (72.0, 41.8), turned to 180 degrees
- moved C22 264.0 mm to (73.0, 75.4), turned to 180 degrees
- moved R14 262.5 mm to (73.0, 69.7), turned to 180 degrees
- moved R15 260.7 mm to (73.0, 79.1), turned to 180 degrees
- moved CR2 258.8 mm to (73.0, 72.5), turned to 180 degrees
- moved R20 257.0 mm to (34.2, 68.5), turned to 270 degrees
- moved SJ3 256.7 mm to (85.6, 65.3)
- moved TP2 255.0 mm to (36.6, 80.3)
- moved C26 254.5 mm to (32.4, 68.5), turned to 270 degrees
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Connections:
- net GPS_USB_DM renamed GPS_USB_N
- net GPS_USB_DP renamed GPS_USB_P
- net SER_DN renamed SER_D_N
- net SER_DP renamed SER_D_P
- new net ADC_VSTORAGE: JP22.1, R10.2, R9.1
- new net MCU_GPS_EN: JP21.2, JP21.3, U3.7
- net 5V: now also C24.1, U6.20
- net GPS_EN: now also JP21.1; no longer U3.7
- net MCU_ADC_VSTORAGE: now also JP22.2, JP22.3, U3.6; no longer R10.2, R9.1
- net N$15: now also R16.1; no longer R13.1
- net N$16: now also R13.1; no longer R16.1
- net USBC_DN: now also CR2.3; no longer CR2.1
- net USBC_DP: now also CR2.1; no longer CR2.3
- net USBC_VBUS: no longer C24.1, U6.20
Routing:
- net GND: track 0.00 -> 137.9 mm, vias 0 -> 106
- net MCU_RESET: track 0.00 -> 107.0 mm, vias 0 -> 4
- net USBC_VBUS: track 0.00 -> 94.4 mm, vias 0 -> 2
- net 5V: track 0.00 -> 90.8 mm, vias 0 -> 4
- net GPS_USB_VDD: track 0.00 -> 81.4 mm, vias 0 -> 2
- net RADIO_GPIO1: track 0.00 -> 67.0 mm, vias 0 -> 1
- net VSOLAR: track 0.00 -> 66.0 mm
- net RADIO_NIRQ: track 0.00 -> 62.4 mm, vias 0 -> 1
- net GPS_USB_P: track 0.00 -> 61.6 mm, vias 0 -> 2
- net N$11: track 0.00 -> 60.3 mm, vias 0 -> 2
- net GPS_USB_N: track 0.00 -> 60.1 mm, vias 0 -> 2
- net SWDIO: track 0.00 -> 59.3 mm, vias 0 -> 1
- net RADIO_EN: track 0.00 -> 57.8 mm, vias 0 -> 2
- net SWCLK: track 0.00 -> 57.6 mm, vias 0 -> 1
- net RADIO_NSS: track 0.00 -> 57.5 mm
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- added copper zone on layer 15, net 3.3V
- added copper zone on layer 1, net GND
- added copper zone on layer 16, net GND
- added copper zone on layer 2, net GND
- added copper zone on layer 1, net GNDKEEPOUT
- added copper zone on layer 15, net GNDKEEPOUT
- added copper zone on layer 16, net GNDKEEPOUT
- added copper zone on layer 2, net GNDKEEPOUT
- added copper zone on layer 15, net VCC
Other:
- board size 160 x 100 mm -> 88.9 x 88.9 mm
- board text added: "HABEXpico Dev Board By: Arko"
